File: Eagle/TurquoiseBicuspid.sch (EAGLE design)
At the start: 14 parts, among them J0 0Ω

Commit message: board v1.1
Parts:
- added J1, J2: 0Ω, rcl:R-US_R1206
Connections:
- net N$23 renamed BT_TX
- removed net N$1: ATTINY85-20SU.PB0, R3.2
- removed net N$2: ATTINY85-20SU.PB1, R2.2
- removed net N$3: ATTINY85-20SU.PB4, R1.2
- removed net N$5: ATTINY85-20SU.PB3, HM-10.UART_RX
- removed net N$7: R3.1, U$1.A3
- removed net N$8: R2.1, U$1.A2
- removed net N$9: R1.1, U$1.A1
- new net A1: ATTINY85-20SU.PB4, R1.1, R1.2, U$1.A1
- new net A2: ATTINY85-20SU.PB1, R2.1, R2.2, U$1.A2
- new net A3: ATTINY85-20SU.PB0, R3.1, R3.2, U$1.A3
- new net BT_RX: ATTINY85-20SU.PB3, HM-10.UART_RX, J1.1, J1.2
- new net RESET: ATTINY85-20SU.NRES/PB5, J2.1, J2.2, R4.2, S1.S, S2.S, S3.S
- net 5V: now also 3.3VREG.EN; no longer ATTINY85-20SU.NRES/PB5, R4.2, S1.S, S2.S, S3.S
Other:
- moved on the sheet: R4
Changed lines of the file:
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@@
 <part name="S3" library="switch-omron" deviceset="10-XX" device=""/>
 <part name="J0" library="rcl" deviceset="R-US_" device="R1206" value="0Ω"/>
+<part name="J1" library="rcl" deviceset="R-US_" device="R1206" value="0Ω"/>
+<part name="J2" library="rcl" deviceset="R-US_" device="R1206" value="0Ω"/>
 </parts>
 <sheets>
@@
 <instance part="R3" gate="G$1" x="15.24" y="2.54" rot="R90"/>
 <instance part="S1" gate="1" x="38.1" y="50.8" rot="R180"/>
-<instance part="R4" gate="G$1" x="66.04" y="43.18"/>
+<instance part="R4" gate="G$1" x="25.4" y="35.56"/>
 <instance part="S2" gate="1" x="45.72" y="50.8" rot="R180"/>
 <instance part="S3" gate="1" x="53.34" y="50.8" rot="R180"/>
 <instance part="J0" gate="G$1" x="33.02" y="-17.78" rot="R90"/>
+<instance part="J1" gate="G$1" x="33.02" y="20.32" rot="R270"/>
+<instance part="J2" gate="G$1" x="35.56" y="38.1" rot="R90"/>
 </instances>
 <busses>
@@
 <net name="5V" class="0">
 <segment>
-<wire x1="-15.24" y1="66.04" x2="30.48" y2="66.04" width="0.1524" layer="91"/>
-<wire x1="30.48" y1="66.04" x2="71.12" y2="66.04" width="0.1524" layer="91"/>
-<wire x1="71.12" y1="43.18" x2="71.12" y2="66.04" width="0.1524" layer="91"/>
-<pinref part="R4" gate="G$1" pin="2"/>
+<wire x1="-15.24" y1="60.96" x2="17.78" y2="60.96" width="0.1524" layer="91"/>
 <pinref part="ATTINY85-20SU" gate="G$1" pin="VCC"/>
 <wire x1="-15.24" y1="22.86" x2="-15.24" y2="25.4" width="0.1524" layer="91"/>
-<wire x1="-15.24" y1="66.04" x2="-15.24" y2="22.86" width="0.1524" layer="91"/>
-<junction x="30.48" y="66.04"/>
-<pinref part="ATTINY85-20SU" gate="G$1" pin="NRES/PB5"/>
-<wire x1="35.56" y1="35.56" x2="35.56" y2="43.18" width="0.1524" layer="91"/>
-<wire x1="35.56" y1="35.56" x2="30.48" y2="35.56" width="0.1524" layer="91"/>
-<wire x1="30.48" y1="35.56" x2="17.78" y2="35.56" width="0.1524" layer="91"/>
-<wire x1="17.78" y1="35.56" x2="17.78" y2="22.86" width="0.1524" layer="91"/>
+<wire x1="-15.24" y1="60.96" x2="-15.24" y2="22.86" width="0.1524" layer="91"/>
 <pinref part="R4" gate="G$1" pin="1"/>
-<wire x1="60.96" y1="43.18" x2="53.34" y2="43.18" width="0.1524" layer="91"/>
-<wire x1="53.34" y1="43.18" x2="45.72" y2="43.18" width="0.1524" layer="91"/>
-<wire x1="45.72" y1="43.18" x2="38.1" y2="43.18" width="0.1524" layer="91"/>
-<pinref part="S2" gate="1" pin="S"/>
-<wire x1="38.1" y1="43.18" x2="35.56" y2="43.18" width="0.1524" layer="91"/>
-<wire x1="45.72" y1="43.18" x2="45.72" y2="45.72" width="0.1524" layer="91"/>
-<pinref part="S3" gate="1" pin="S"/>
-<wire x1="53.34" y1="43.18" x2="53.34" y2="45.72" width="0.1524" layer="91"/>
-<junction x="53.34" y="43.18"/>
-<junction x="45.72" y="43.18"/>
-<pinref part="S1" gate="1" pin="S"/>
-<wire x1="38.1" y1="45.72" x2="38.1" y2="43.18" width="0.1524" layer="91"/>
-<junction x="38.1" y="43.18"/>
-<junction x="30.48" y="35.56"/>
-<wire x1="30.48" y1="66.04" x2="30.48" y2="35.56" width="0.1524" layer="91"/>
+<wire x1="17.78" y1="35.56" x2="17.78" y2="60.96" width="0.1524" layer="91"/>
+<wire x1="20.32" y1="35.56" x2="17.78" y2="35.56" width="0.1524" layer="91"/>
 </segment>
 <segment>
@@
 <wire x1="-40.64" y1="22.86" x2="-40.64" y2="43.18" width="0.1524" layer="91"/>
 <wire x1="-40.64" y1="43.18" x2="-15.24" y2="43.18" width="0.1524" layer="91"/>
+<pinref part="3.3VREG" gate="G1" pin="EN"/>
+<wire x1="-10.16" y1="40.64" x2="-12.7" y2="40.64" width="0.1524" layer="91"/>
+<wire x1="-12.7" y1="40.64" x2="-12.7" y2="43.18" width="0.1524" layer="91"/>
+<junction x="-12.7" y="43.18"/>
 </segment>
 </net>
@@
 </segment>
 </net>
-<net name="N$1" class="0">
+<net name="A3" class="0">
 <segment>
 <pinref part="ATTINY85-20SU" gate="G$1" pin="PB0"/>
@@
 <pinref part="R3" gate="G$1" pin="2"/>
 </segment>
-</net>
-<net name="N$2" class="0">
+<segment>
+<pinref part="U$1" gate="G$1" pin="A3"/>
+<wire x1="15.24" y1="-5.08" x2="10.16" y2="-5.08" width="0.1524" layer="91"/>
+<pinref part="R3" gate="G$1" pin="1"/>
+<wire x1="15.24" y1="-5.08" x2="15.24" y2="-2.54" width="0.1524" layer="91"/>
+</segment>
+</net>
+<net name="A2" class="0">
 <segment>
 <pinref part="ATTINY85-20SU" gate="G$1" pin="PB1"/>
@@
 <pinref part="R2" gate="G$1" pin="2"/>
 </segment>
-</net>
-<net name="N$3" class="0">
-<segment>
-<pinref part="ATTINY85-20SU" gate="G$1" pin="PB4"/>
-<wire x1="17.78" y1="20.32" x2="22.86" y2="20.32" width="0.1524" layer="91"/>
-<wire x1="22.86" y1="20.32" x2="22.86" y2="2.54" width="0.1524" layer="91"/>
-<wire x1="22.86" y1="2.54" x2="20.32" y2="2.54" width="0.1524" layer="91"/>
-<pinref part="R1" gate="G$1" pin="2"/>
+<segment>
+<pinref part="U$1" gate="G$1" pin="A2"/>
+<wire x1="17.78" y1="-7.62" x2="15.24" y2="-7.62" width="0.1524" layer="91"/>
+<wire x1="15.24" y1="-7.62" x2="15.24" y2="-10.16" width="0.1524" layer="91"/>
+<wire x1="15.24" y1="-10.16" x2="10.16" y2="-10.16" width="0.1524" layer="91"/>
+<pinref part="R2" gate="G$1" pin="1"/>
+<wire x1="17.78" y1="-7.62" x2="17.78" y2="-5.08" width="0.1524" layer="91"/>
 </segment>
 </net>
@@
 </segment>
 </net>
-<net name="N$7" class="0">
-<segment>
-<pinref part="U$1" gate="G$1" pin="A3"/>
-<wire x1="15.24" y1="-5.08" x2="10.16" y2="-5.08" width="0.1524" layer="91"/>
-<pinref part="R3" gate="G$1" pin="1"/>
-<wire x1="15.24" y1="-5.08" x2="15.24" y2="-2.54" width="0.1524" layer="91"/>
-</segment>
-</net>
-<net name="N$8" class="0">
-<segment>
-<pinref part="U$1" gate="G$1" pin="A2"/>
-<wire x1="17.78" y1="-7.62" x2="15.24" y2="-7.62" width="0.1524" layer="91"/>
-<wire x1="15.24" y1="-7.62" x2="15.24" y2="-10.16" width="0.1524" layer="91"/>
-<wire x1="15.24" y1="-10.16" x2="10.16" y2="-10.16" width="0.1524" layer="91"/>
-<pinref part="R2" gate="G$1" pin="1"/>
-<wire x1="17.78" y1="-7.62" x2="17.78" y2="-5.08" width="0.1524" layer="91"/>
-</segment>
-</net>
-<net name="N$9" class="0">
+<net name="A1" class="0">
 <segment>
 <pinref part="U$1" gate="G$1" pin="A1"/>
@@
 <wire x1="20.32" y1="-10.16" x2="20.32" y2="-7.62" width="0.1524" layer="91"/>
 </segment>
+<segment>
+<pinref part="ATTINY85-20SU" gate="G$1" pin="PB4"/>
+<wire x1="17.78" y1="20.32" x2="22.86" y2="20.32" width="0.1524" layer="91"/>
+<wire x1="22.86" y1="20.32" x2="22.86" y2="2.54" width="0.1524" layer="91"/>
+<wire x1="22.86" y1="2.54" x2="20.32" y2="2.54" width="0.1524" layer="91"/>
+<pinref part="R1" gate="G$1" pin="2"/>
+</segment>
 </net>
 <net name="N$6" class="0">
@@
 </segment>
 </net>
-<net name="N$23" class="0">
+<net name="BT_TX" class="0">
 <segment>
 <pinref part="HM-10" gate="G$1" pin="UART_TX"/>
@@
 </segment>
 </net>
-<net name="N$5" class="0">
-<segment>
-<pinref part="HM-10" gate="G$1" pin="UART_RX"/>
-<wire x1="35.56" y1="25.4" x2="30.48" y2="25.4" width="0.1524" layer="91"/>
-<wire x1="30.48" y1="25.4" x2="30.48" y2="17.78" width="0.1524" layer="91"/>
+<net name="BT_RX" class="0">
+<segment>
 <pinref part="ATTINY85-20SU" gate="G$1" pin="PB3"/>
 <wire x1="30.48" y1="17.78" x2="17.78" y2="17.78" width="0.1524" layer="91"/>
-</segment>
-</net>
+<pinref part="J1" gate="G$1" pin="2"/>
+<wire x1="33.02" y1="15.24" x2="30.48" y2="15.24" width="0.1524" layer="91"/>
+<wire x1="30.48" y1="15.24" x2="30.48" y2="17.78" width="0.1524" layer="91"/>
+</segment>
+<segment>
+<pinref part="HM-10" gate="G$1" pin="UART_RX"/>
+<wire x1="35.56" y1="25.4" x2="33.02" y2="25.4" width="0.1524" layer="91"/>
+<pinref part="J1" gate="G$1" pin="1"/>
+</segment>
+</net>
+<net name="RESET" class="0">
+<segment>
+<wire x1="33.02" y1="35.56" x2="30.48" y2="35.56" width="0.1524" layer="91"/>
+<pinref part="R4" gate="G$1" pin="2"/>
+<pinref part="ATTINY85-20SU" gate="G$1" pin="NRES/PB5"/>
+<wire x1="17.78" y1="22.86" x2="17.78" y2="30.48" width="0.1524" layer="91"/>
+<wire x1="17.78" y1="30.48" x2="33.02" y2="30.48" width="0.1524" layer="91"/>
+<wire x1="33.02" y1="30.48" x2="33.02" y2="35.56" width="0.1524" layer="91"/>
+<wire x1="33.02" y1="30.48" x2="35.56" y2="30.48" width="0.1524" layer="91"/>
+<pinref part="J2" gate="G$1" pin="1"/>
+<wire x1="35.56" y1="30.48" x2="35.56" y2="33.02" width="0.1524" layer="91"/>
+</segment>
+<segment>
+<pinref part="S2" gate="1" pin="S"/>
+<pinref part="S3" gate="1" pin="S"/>
+<wire x1="53.34" y1="43.18" x2="53.34" y2="45.72" width="0.1524" layer="91"/>
+<wire x1="53.34" y1="43.18" x2="45.72" y2="43.18" width="0.1524" layer="91"/>
+<wire x1="45.72" y1="43.18" x2="45.72" y2="45.72" width="0.1524" layer="91"/>
+<junction x="45.72" y="43.18"/>
+<wire x1="45.72" y1="43.18" x2="38.1" y2="43.18" width="0.1524" layer="91"/>
+<pinref part="S1" gate="1" pin="S"/>
+<wire x1="38.1" y1="45.72" x2="38.1" y2="43.18" width="0.1524" layer="91"/>
+<junction x="38.1" y="43.18"/>
+<wire x1="38.1" y1="43.18" x2="35.56" y2="43.18" width="0.1524" layer="91"/>
+<pinref part="J2" gate="G$1" pin="2"/>
+</segment>
+</net>
